File: inputs.kicad_sch (KiCad schematic)
At the start: 64 parts, among them J10 IN6, J11 IN7, J12 IN8, J5 IN1, J6 IN2, J7 IN3, J8 IN4, J9 IN5, U10 EL357N, U11 EL357N, U4 EL357N, U5 EL357N, U6 EL357N, U7 EL357N, U8 EL357N, U9 EL357N

Commit message: Add real footprints (HK4100F/AQY212GS/EL357N) + tidy schematic (rev 0.3)
- Build datasheet-accurate HK4100F-DC5V-SHG footprint (6-pad THT) and a
  matching symbol; coil=3/4, COM=5/6, NO=1, NC=2.
- Correct AQY212GS footprint to SOP-4 2.54mm pitch (was wrongly 1.27mm).
- Fix EL357N LCSC code C124981->C6649 (C124981 was a trimmer pot); add
  generated SOP-4 footprint.
- footprints/bridge.pretty generated from LCSC parts via easyeda2kicad.
- Re-lay-out all sheets for human review: labels offset from pins via
  short stubs routed by each pin's true orientation; 8-channel sheets on
  larger pages; clean per-channel columns.
- ERC still 0 errors / 0 warnings. Regenerated schematic.pdf, BOM, DESIGN.
- No PCB layout yet (paused per request).

Co-Authored-By: Claude Opus 4.7 <noreply@anthropic.com>
Parts:
- U10, U11, U4, U5, U6, U7, U8, U9: footprint Package_SO:SOP-4_4.4x2.6mm_P1.27mm -> bridge:EL357N_SOP-4
Other:
- note added: "Wide-range isolated input x8. R(2.2k/1206)+EL357N+anti-parallel diode + RC filter. Active-LOW."
- note removed: "Wide-range isolated input x8. R(2.2k/1206)+EL357N+anti-parallel diode. RC filter. Active-LOW."
