File: mcu.kicad_sch (KiCad schematic)
At the start: 0 parts

Commit message: Realize ERC-clean KiCad schematic (rev 0.2)
Turn the paper design into a real KiCad 10 hierarchical schematic with
library symbols and footprints. 6 sheets: power, MCU, and full channel
counts (8 inputs, 8 PhotoMOS, 2 relays, 4 cap-inject) = 160 components.

- Replace AMS1117 with SY8089 buck (2.7-5.5Vin) for Wi-Fi-peak headroom.
- Input front-end uses 2.2k/1206 + EL357N (CRD dropped; poor LCSC stock).
- Verify key parts against JLCPCB (ESP32-S3 C2913198, SY8089 C78988,
  AQY212GS C719745, HK4100F C12072, USB-C C165948, AO3400A C20917).
- ERC passes 0 errors / 0 warnings; netlist verified, isolation barrier
  confirmed intact. No PCB layout yet (per request).
- Add Python generator (gen/) that emits the project and custom symbols.

Co-Authored-By: Claude Opus 4.7 <noreply@anthropic.com>
Parts:
- added C5: 1uF, Capacitor_SMD:C_0603_1608Metric, symbol Device:C
- added C6, C7, C8: 100nF, Capacitor_SMD:C_0603_1608Metric, symbol Device:C
- added C9: 10uF, Capacitor_SMD:C_0603_1608Metric, symbol Device:C
- added D3: STATUS, LED_SMD:LED_0603_1608Metric, symbol Device:LED
- added J3: UART, Connector_PinHeader_2.54mm:PinHeader_1x03_P2.54mm_Vertical, symbol Connector_Generic:Conn_01x03
- added J4: SPARE GPIO, Connector_PinHeader_2.54mm:PinHeader_1x06_P2.54mm_Vertical, symbol Connector_Generic:Conn_01x06
- added R5, R6: 10k, Resistor_SMD:R_0603_1608Metric, symbol Device:R
- added R7: 1k, Resistor_SMD:R_0603_1608Metric, symbol Device:R
- added SW1: RESET, Button_Switch_SMD:Panasonic_EVQPUJ_EVQPUA, symbol Switch:SW_Push
- added SW2: BOOT, Button_Switch_SMD:Panasonic_EVQPUJ_EVQPUA, symbol Switch:SW_Push
- added U3: ESP32-S3-WROOM-1-N8, RF_Module:ESP32-S3-WROOM-1, symbol RF_Module:ESP32-S3-WROOM-1
Connections:
- new net +3V3: C7.1, C8.1, C9.1, R5.1, R6.1, U3.2 (3V3)
- new net BOOT_NET: C6.1, R6.2, SW2.1, U3.27 (IO0)
- new net CAP1: U3.30 (IO37)
- new net CAP2: U3.31 (IO38)
- new net CAP3: U3.32 (IO39)
- new net CAP4: U3.33 (IO40)
- new net DBG_RX: J3.2 (Pin_2), U3.36 (RXD0)
- new net DBG_TX: J3.1 (Pin_1), U3.37 (TXD0)
- new net EN_NET: C5.1, R5.2, SW1.1, U3.3 (EN)
- new net GND: C5.2, C6.2, C7.2, C8.2, C9.2, D3.1 (K), J3.3 (Pin_3), J4.6 (Pin_6), SW1.2, SW2.2, U3.1 (GND), U3.40 (GND), U3.41 (GND)
- new net IN1: U3.4 (IO4)
- new net IN2: U3.5 (IO5)
- new net IN3: U3.6 (IO6)
- new net IN4: U3.7 (IO7)
- new net IN5: U3.8 (IO15)
- new net IN6: U3.9 (IO16)
- new net IN7: U3.10 (IO17)
- new net IN8: U3.11 (IO18)
- new net LEDNET: R7.1, U3.38 (IO2)
- new net LED_AK: D3.2 (A), R7.2
- new net OUT1: U3.12 (IO8)
- new net OUT2: U3.17 (IO9)
- new net OUT3: U3.18 (IO10)
- new net OUT4: U3.19 (IO11)
- new net OUT5: U3.20 (IO12)
- new net OUT6: U3.21 (IO13)
- new net OUT7: U3.22 (IO14)
- new net OUT8: U3.23 (IO21)
- new net RLY1: U3.28 (IO35)
- new net RLY2: U3.29 (IO36)
- new net SP_24: J4.1 (Pin_1), U3.24 (IO47)
- new net SP_25: J4.2 (Pin_2), U3.25 (IO48)
- new net SP_34: J4.3 (Pin_3), U3.34 (IO41)
- new net SP_35: J4.4 (Pin_4), U3.35 (IO42)
- new net SP_39: J4.5 (Pin_5), U3.39 (IO1)
- new net USB_D+: U3.14 (USB_D+)
- new net USB_D-: U3.13 (USB_D-)
- no-connect marks 0 -> 3
Other:
- removed sheet CapInject
- removed sheet Inputs
- removed sheet MCU
- removed sheet PhotoMOS
- removed sheet Power
- removed sheet Relays
- note added: "ESP32-S3-WROOM-1-N8. Strapping IO3/45/46=NC. IO0=BOOT, EN=RESET. Native USB IO19/20. Status LED IO2."
- title: Universal ESP32 Button/Signal Bridge -> ESP32-S3-WROOM-1-N8
