File: photomos.kicad_sch (KiCad schematic)
At the start: 0 parts

Commit message: Realize ERC-clean KiCad schematic (rev 0.2)
Turn the paper design into a real KiCad 10 hierarchical schematic with
library symbols and footprints. 6 sheets: power, MCU, and full channel
counts (8 inputs, 8 PhotoMOS, 2 relays, 4 cap-inject) = 160 components.

- Replace AMS1117 with SY8089 buck (2.7-5.5Vin) for Wi-Fi-peak headroom.
- Input front-end uses 2.2k/1206 + EL357N (CRD dropped; poor LCSC stock).
- Verify key parts against JLCPCB (ESP32-S3 C2913198, SY8089 C78988,
  AQY212GS C719745, HK4100F C12072, USB-C C165948, AO3400A C20917).
- ERC passes 0 errors / 0 warnings; netlist verified, isolation barrier
  confirmed intact. No PCB layout yet (per request).
- Add Python generator (gen/) that emits the project and custom symbols.

Co-Authored-By: Claude Opus 4.7 <noreply@anthropic.com>
Parts:
- added J13: OUT1, TerminalBlock:TerminalBlock_MaiXu_MX126-5.0-02P_1x02_P5.00mm, symbol Connector_Generic:Conn_01x02
- added J14: OUT2, TerminalBlock:TerminalBlock_MaiXu_MX126-5.0-02P_1x02_P5.00mm, symbol Connector_Generic:Conn_01x02
- added J15: OUT3, TerminalBlock:TerminalBlock_MaiXu_MX126-5.0-02P_1x02_P5.00mm, symbol Connector_Generic:Conn_01x02
- added J16: OUT4, TerminalBlock:TerminalBlock_MaiXu_MX126-5.0-02P_1x02_P5.00mm, symbol Connector_Generic:Conn_01x02
- added J17: OUT5, TerminalBlock:TerminalBlock_MaiXu_MX126-5.0-02P_1x02_P5.00mm, symbol Connector_Generic:Conn_01x02
- added J18: OUT6, TerminalBlock:TerminalBlock_MaiXu_MX126-5.0-02P_1x02_P5.00mm, symbol Connector_Generic:Conn_01x02
- added J19: OUT7, TerminalBlock:TerminalBlock_MaiXu_MX126-5.0-02P_1x02_P5.00mm, symbol Connector_Generic:Conn_01x02
- added J20: OUT8, TerminalBlock:TerminalBlock_MaiXu_MX126-5.0-02P_1x02_P5.00mm, symbol Connector_Generic:Conn_01x02
- added R32, R33, R34, R35, R36, R37, R38, R39: 330, Resistor_SMD:R_0603_1608Metric, symbol Device:R
- added TP12: OUT1, TestPoint:TestPoint_Pad_D1.5mm, symbol Connector:TestPoint
- added TP13: OUT2, TestPoint:TestPoint_Pad_D1.5mm, symbol Connector:TestPoint
- added TP14: OUT3, TestPoint:TestPoint_Pad_D1.5mm, symbol Connector:TestPoint
- added TP15: OUT4, TestPoint:TestPoint_Pad_D1.5mm, symbol Connector:TestPoint
- added TP16: OUT5, TestPoint:TestPoint_Pad_D1.5mm, symbol Connector:TestPoint
- added TP17: OUT6, TestPoint:TestPoint_Pad_D1.5mm, symbol Connector:TestPoint
- added TP18: OUT7, TestPoint:TestPoint_Pad_D1.5mm, symbol Connector:TestPoint
- added TP19: OUT8, TestPoint:TestPoint_Pad_D1.5mm, symbol Connector:TestPoint
- added U12, U13, U14, U15, U16, U17, U18, U19: AQY212GS, Package_SO:SOP-4_4.4x2.6mm_P1.27mm, symbol bridge:AQY212GS
Connections:
- new net GND: U12.2 (K), U13.2 (K), U14.2 (K), U15.2 (K), U16.2 (K), U17.2 (K), U18.2 (K), U19.2 (K)
- new net OUT1: R32.1
- new net OUT1_A: J13.1 (Pin_1), TP12.1, U12.4 (L1)
- new net OUT1_B: J13.2 (Pin_2), U12.3 (L2)
- new net OUT1_LED: R32.2, U12.1 (A)
- new net OUT2: R33.1
- new net OUT2_A: J14.1 (Pin_1), TP13.1, U13.4 (L1)
- new net OUT2_B: J14.2 (Pin_2), U13.3 (L2)
- new net OUT2_LED: R33.2, U13.1 (A)
- new net OUT3: R34.1
- new net OUT3_A: J15.1 (Pin_1), TP14.1, U14.4 (L1)
- new net OUT3_B: J15.2 (Pin_2), U14.3 (L2)
- new net OUT3_LED: R34.2, U14.1 (A)
- new net OUT4: R35.1
- new net OUT4_A: J16.1 (Pin_1), TP15.1, U15.4 (L1)
- new net OUT4_B: J16.2 (Pin_2), U15.3 (L2)
- new net OUT4_LED: R35.2, U15.1 (A)
- new net OUT5: R36.1
- new net OUT5_A: J17.1 (Pin_1), TP16.1, U16.4 (L1)
- new net OUT5_B: J17.2 (Pin_2), U16.3 (L2)
- new net OUT5_LED: R36.2, U16.1 (A)
- new net OUT6: R37.1
- new net OUT6_A: J18.1 (Pin_1), TP17.1, U17.4 (L1)
- new net OUT6_B: J18.2 (Pin_2), U17.3 (L2)
- new net OUT6_LED: R37.2, U17.1 (A)
- new net OUT7: R38.1
- new net OUT7_A: J19.1 (Pin_1), TP18.1, U18.4 (L1)
- new net OUT7_B: J19.2 (Pin_2), U18.3 (L2)
- new net OUT7_LED: R38.2, U18.1 (A)
- new net OUT8: R39.1
- new net OUT8_A: J20.1 (Pin_1), TP19.1, U19.4 (L1)
- new net OUT8_B: J20.2 (Pin_2), U19.3 (L2)
- new net OUT8_LED: R39.2, U19.1 (A)
Other:
- removed sheet CapInject
- removed sheet Inputs
- removed sheet MCU
- removed sheet PhotoMOS
- removed sheet Power
- removed sheet Relays
- note added: "PhotoMOS isolated dry contact x8. GPIO->330R->AQY212GS. HIGH=closed. <=60V/<=0.5A."
- title: Universal ESP32 Button/Signal Bridge -> 8x PhotoMOS dry-contact outputs

Commit message: Add real footprints (HK4100F/AQY212GS/EL357N) + tidy schematic (rev 0.3)
- Build datasheet-accurate HK4100F-DC5V-SHG footprint (6-pad THT) and a
  matching symbol; coil=3/4, COM=5/6, NO=1, NC=2.
- Correct AQY212GS footprint to SOP-4 2.54mm pitch (was wrongly 1.27mm).
- Fix EL357N LCSC code C124981->C6649 (C124981 was a trimmer pot); add
  generated SOP-4 footprint.
- footprints/bridge.pretty generated from LCSC parts via easyeda2kicad.
- Re-lay-out all sheets for human review: labels offset from pins via
  short stubs routed by each pin's true orientation; 8-channel sheets on
  larger pages; clean per-channel columns.
- ERC still 0 errors / 0 warnings. Regenerated schematic.pdf, BOM, DESIGN.
- No PCB layout yet (paused per request).

Co-Authored-By: Claude Opus 4.7 <noreply@anthropic.com>
Parts:
- U12, U13, U14, U15, U16, U17, U18, U19: footprint Package_SO:SOP-4_4.4x2.6mm_P1.27mm -> bridge:AQY212GS_SOP-4
