File: power.kicad_sch (KiCad schematic)
At the start: 0 parts

Commit message: Realize ERC-clean KiCad schematic (rev 0.2)
Turn the paper design into a real KiCad 10 hierarchical schematic with
library symbols and footprints. 6 sheets: power, MCU, and full channel
counts (8 inputs, 8 PhotoMOS, 2 relays, 4 cap-inject) = 160 components.

- Replace AMS1117 with SY8089 buck (2.7-5.5Vin) for Wi-Fi-peak headroom.
- Input front-end uses 2.2k/1206 + EL357N (CRD dropped; poor LCSC stock).
- Verify key parts against JLCPCB (ESP32-S3 C2913198, SY8089 C78988,
  AQY212GS C719745, HK4100F C12072, USB-C C165948, AO3400A C20917).
- ERC passes 0 errors / 0 warnings; netlist verified, isolation barrier
  confirmed intact. No PCB layout yet (per request).
- Add Python generator (gen/) that emits the project and custom symbols.

Co-Authored-By: Claude Opus 4.7 <noreply@anthropic.com>
Parts:
- added C1: 100uF, Capacitor_SMD:C_1206_3216Metric, symbol Device:C
- added C2: 100nF, Capacitor_SMD:C_0603_1608Metric, symbol Device:C
- added C3, C4: 22uF, Capacitor_SMD:C_0805_2012Metric, symbol Device:C
- added D1, D2: SS54, Diode_SMD:D_SMC, symbol Device:D_Schottky
- added J1: USB-C, Connector_USB:USB_C_Receptacle_HRO_TYPE-C-31-M-12, symbol Connector:USB_C_Receptacle_USB2.0_16P
- added J2: EXT 5V, TerminalBlock:TerminalBlock_MaiXu_MX126-5.0-02P_1x02_P5.00mm, symbol Connector_Generic:Conn_01x02
- added L1: 2.2uH, Inductor_SMD:L_1210_3225Metric, symbol Device:L
- added R1, R2: 5.1k, Resistor_SMD:R_0603_1608Metric, symbol Device:R
- added R3: 453k, Resistor_SMD:R_0603_1608Metric, symbol Device:R
- added R4: 100k, Resistor_SMD:R_0603_1608Metric, symbol Device:R
- added TP1: +5V, TestPoint:TestPoint_Pad_D1.5mm, symbol Connector:TestPoint
- added TP2: +3V3, TestPoint:TestPoint_Pad_D1.5mm, symbol Connector:TestPoint
- added TP3: GND, TestPoint:TestPoint_Pad_D1.5mm, symbol Connector:TestPoint
- added U1: USBLC6-2SC6, Package_TO_SOT_SMD:SOT-23-6, symbol Power_Protection:USBLC6-2P6
- added U2: SY8089AAAC, Package_TO_SOT_SMD:SOT-23-5, symbol bridge:SY8089
Connections:
- new net +3V3: C4.1, L1.2, R3.1, TP2.1
- new net +5V: C1.1, C2.1, C3.1, D1.1 (K), D2.1 (K), TP1.1, U2.1 (EN), U2.4 (IN)
- new net CC1: J1.A5 (CC1), R1.1
- new net CC2: J1.B5 (CC2), R2.1
- new net EXT5V: D2.2 (A), J2.1 (Pin_1)
- new net FB: R3.2, R4.1, U2.5 (FB)
- new net GND: C1.2, C2.2, C3.2, C4.2, J1.A1 (GND), J1.A12 (GND), J1.B1 (GND), J1.B12 (GND), J1.SH (SHIELD), J2.2 (Pin_2), R1.2, R2.2, R4.2, TP3.1, U1.2 (GND), U2.2 (GND)
- new net SW: L1.1, U2.3 (LX)
- new net USB_D+: U1.6 (I/O1)
- new net USB_D-: U1.4 (I/O2)
- new net USB_DM_RAW: J1.A7 (D-), J1.B7 (D-), U1.3 (I/O2)
- new net USB_DP_RAW: J1.A6 (D+), J1.B6 (D+), U1.1 (I/O1)
- new net VBUS: D1.2 (A), J1.A4 (VBUS), J1.A9 (VBUS), J1.B4 (VBUS), J1.B9 (VBUS), U1.5 (VBUS)
- no-connect marks 0 -> 2
Other:
- removed sheet CapInject
- removed sheet Inputs
- removed sheet MCU
- removed sheet PhotoMOS
- removed sheet Power
- removed sheet Relays
- note added: "USB-C diode-OR -> SY8089 buck (2.7-5.5Vin,2A) -> 3.3V. EN tied +5V. Vout=0.6*(1+R/R)=3.32V."
- title: Universal ESP32 Button/Signal Bridge -> Power - USB-C / diode-OR / SY8089 buck 3.3V

Commit message: Add real footprints (HK4100F/AQY212GS/EL357N) + tidy schematic (rev 0.3)
- Build datasheet-accurate HK4100F-DC5V-SHG footprint (6-pad THT) and a
  matching symbol; coil=3/4, COM=5/6, NO=1, NC=2.
- Correct AQY212GS footprint to SOP-4 2.54mm pitch (was wrongly 1.27mm).
- Fix EL357N LCSC code C124981->C6649 (C124981 was a trimmer pot); add
  generated SOP-4 footprint.
- footprints/bridge.pretty generated from LCSC parts via easyeda2kicad.
- Re-lay-out all sheets for human review: labels offset from pins via
  short stubs routed by each pin's true orientation; 8-channel sheets on
  larger pages; clean per-channel columns.
- ERC still 0 errors / 0 warnings. Regenerated schematic.pdf, BOM, DESIGN.
- No PCB layout yet (paused per request).

Co-Authored-By: Claude Opus 4.7 <noreply@anthropic.com>
Other:
- note added: "USB-C diode-OR -> SY8089 buck (2.7-5.5Vin,2A) -> 3.3V. EN tied +5V. Vout=0.6*(1+R3/R4)=3.32V."
- note removed: "USB-C diode-OR -> SY8089 buck (2.7-5.5Vin,2A) -> 3.3V. EN tied +5V. Vout=0.6*(1+R/R)=3.32V."
